File: hello.sch (KiCad schematic (older format))
At the start: 50 parts, among them J1 USB_OTG, J2 Conn_02x05_Odd_Even, J3 Conn_01x07, J4 Conn_01x04, Q1 DMG1012UW, Q2 DMG1012UW, Q3 DMG1012UW, Q4 DMG1012UW, Q5 DMG1012UW, Q6 NTR1P02T1G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

Commit message: Fix pinout for BAS116 diode (D3)
Parts:
- D3: symbol D_Small_ALT -> BAS116
Connections:
- net VBUS: now also D3.1 (A); no longer D3.2 (A)
- net at C11.1, Q6.2 (S), SW2.3 (C)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: now also D3.3 (K); no longer D3.1 (K)
Changed lines of the file:
@@
 $EndComp
 $Comp
-L D_Small_ALT D3
+L BAS116 D3
 U 1 1 5CD7602C
 P 9500 1150
